File: CPLD_bcdtohex.kicad_sch (KiCad schematic)
At the start: 25 parts, among them IC1 ATF750C-10PU, SW1 SW_DIP_x06

Commit message: Initial commit
Parts:
- removed SW1: SW_DIP_x06, Button_Switch_THT:SW_DIP_SPSTx06_Slide_9.78x17.42mm_W7.62mm_P2.54mm, symbol Switch:SW_DIP_x06
- added J1: Conn_01x06, symbol Connector_Generic:Conn_01x06
- added J2: Conn_01x02, symbol Connector_Generic:Conn_01x02
Connections:
- net +5V: now also J2.1 (Pin_1)
- net GND: now also R5.2, R6.2, J2.2 (Pin_2); no longer R5.1, R6.1
- net at IC1.4 (IN_3), R16.1, R2.2: now also J1.2 (Pin_2)
- net at IC1.6 (IN_5): now also R5.1, J1.5 (Pin_5); no longer R5.2
- net at IC1.2 (IN_1), R18.1, R4.2: now also J1.4 (Pin_4)
- net at IC1.3 (IN_2), R17.1, R3.2: now also J1.3 (Pin_3)
- net at IC1.5 (IN_4), R1.2, R15.1: now also J1.1 (Pin_1)
- net at IC1.7 (IN_6): now also R6.1, J1.6 (Pin_6); no longer R6.2
Other:
- moved on the sheet: D1, D2, D3, D4, DS1, IC1, R1, R10, R11, R12, R13, R14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
