File: CPLD_bcdtohex.kicad_sch (KiCad schematic)
At the start: 26 parts, among them IC1 ATF750C-10PU, J1 Conn_01x06, J2 Conn_01x02

Commit message: Initial commit
Parts:
- removed D1, D2, D3, D4: LED, LED_THT:LED_D5.0mm, symbol Device:LED
- removed R1, R2, R3, R4, R5, R6: 10k, Resistor_THT:R_Axial_DIN0204_L3.6mm_D1.6mm_P5.08mm_Horizontal, symbol Device:R_US
- removed R10, R11, R12, R13, R14, R7, R8, R9: 330, Resistor_THT:R_Axial_DIN0204_L3.6mm_D1.6mm_P5.08mm_Horizontal, symbol Device:R_US
- removed R15, R16, R17, R18: 220, Resistor_THT:R_Axial_DIN0204_L3.6mm_D1.6mm_P5.08mm_Horizontal, symbol Device:R_US
- added RN1: 12K, Resistor_THT:R_Array_SIP7, symbol Device:R_Network06
- added RN2: 330, Package_DIP:DIP-16_W7.62mm, symbol Device:R_Pack08
- IC1: footprint Package_DIP:DIP-24_W15.24mm -> Package_DIP:DIP-24_W10.16mm
- J1: footprint (none) -> Connector_PinHeader_2.54mm:PinHeader_1x06_P2.54mm_Vertical
- J2: footprint (none) -> Connector_PinHeader_2.54mm:PinHeader_1x02_P2.54mm_Vertical
Connections:
- net GND: now also RN1.1 (common)
- net bit1_in: now reaches IC1.4 (IN_3)
- net bit1_in: now also J1.3 (Pin_3), RN1.4 (R3); no longer J1.2 (Pin_2)
- net at IC1.21 (I/O_8): now also RN2.9 (R8.2)
- net a: now reaches DS1.10 (a)
- net a: now also RN2.8 (R8.1)
- net BLANK_in: now reaches IC1.6 (IN_5), J1.5 (Pin_5)
- net BLANK_in: now also RN1.6 (R5)
- net bit0_in: now reaches J1.4 (Pin_4)
- net bit0_in: now also IC1.5 (IN_4), RN1.5 (R4); no longer IC1.2 (IN_1)
- net g: now reaches DS1.1 (g)
- net g: now also RN2.2 (R2.1)
- net f: now reaches DS1.2 (f)
- net f: now also RN2.3 (R3.1)
- net e: now reaches DS1.4 (e)
- net e: now also RN2.4 (R4.1)
- net d: now reaches DS1.5 (d)
- net d: now also RN2.5 (R5.1)
- net dp: now reaches DS1.6 (DP)
- net dp: now also RN2.1 (R1.1)
- net c: now reaches DS1.7 (c)
- net c: now also RN2.6 (R6.1)
- net b: now reaches DS1.9 (b)
- net b: now also RN2.7 (R7.1)
- net at IC1.18 (I/O_5): now also RN2.12 (R5.2)
- net at IC1.14 (I/O_1): now also RN2.16 (R1.2)
- net at IC1.15 (I/O_2): now also RN2.15 (R2.2)
- net at IC1.16 (I/O_3): now also RN2.14 (R3.2)
- net at IC1.17 (I/O_4): now also RN2.13 (R4.2)
- net at IC1.19 (I/O_6): now also RN2.11 (R6.2)
- net at IC1.20 (I/O_7): now also RN2.10 (R7.2)
- net bit2_in: now reaches IC1.3 (IN_2)
- net bit2_in: now also J1.2 (Pin_2), RN1.3 (R2); no longer J1.3 (Pin_3)
- net bit3_in: now reaches J1.1 (Pin_1)
- net bit3_in: now also IC1.2 (IN_1), RN1.2 (R1); no longer IC1.5 (IN_4)
- net DP_in: now reaches IC1.7 (IN_6), J1.6 (Pin_6)
- net DP_in: now also RN1.7 (R6)
Other:
- note added: "Inputs"
- note added: "Outputs"
- moved on the sheet: DS1, IC1, J1, J2

Commit message: Initial commit
Parts:
- removed J1: Conn_01x06, Connector_PinHeader_2.54mm:PinHeader_1x06_P2.54mm_Vertical, symbol Connector_Generic:Conn_01x06
- removed J2: Conn_01x02, Connector_PinHeader_2.54mm:PinHeader_1x02_P2.54mm_Vertical, symbol Connector_Generic:Conn_01x02
- added J1: Conn_01x08_Pin, symbol Connector:Conn_01x08_Pin
Connections:
- net +5V: now also J1.1 (Pin_1)
- net BLANK_in: now also J1.7 (Pin_7)
- net DP_in: now also J1.8 (Pin_8)
- net GND: now also J1.2 (Pin_2)
- net bit0_in: now also J1.6 (Pin_6)
- net bit1_in: now also J1.5 (Pin_5)
- net bit2_in: now also J1.4 (Pin_4)
- net bit3_in: now also J1.3 (Pin_3)
Other:
- moved on the sheet: RN1

Commit message: Initial commit
Parts:
- J1: footprint (none) -> Connector_PinHeader_2.54mm:PinHeader_1x08_P2.54mm_Vertical
Connections:
- net bit2_in is gone; now on net BIT2_IN: IC1.3 (IN_2), J1.4 (Pin_4), RN1.3 (R2)
- net DP_OUT_N: now reaches IC1.14 (I/O_1), RN2.16 (R1.2)
- net SEG_G_OUT_N: now reaches IC1.15 (I/O_2), RN2.15 (R2.2)
- net SEG_F_OUT_N: now reaches IC1.16 (I/O_3), RN2.14 (R3.2)
- net SEG_E_OUT_N: now reaches IC1.17 (I/O_4), RN2.13 (R4.2)
- net SEG_D_OUT_N: now reaches IC1.18 (I/O_5), RN2.12 (R5.2)
- net SEG_C_OUT_N: now reaches IC1.19 (I/O_6), RN2.11 (R6.2)
- net SEG_B_OUT_N: now reaches IC1.20 (I/O_7), RN2.10 (R7.2)
- net SEG_A_OUT_N: now reaches IC1.21 (I/O_8), RN2.9 (R8.2)
- net BLANK_in renamed BLANK_IN_N
- net DP_in renamed DP_IN
- net a: no longer names the net of DS1.10 (a), RN2.8 (R8.1)
- net b: no longer names the net of DS1.9 (b), RN2.7 (R7.1)
- net bit0_in renamed BIT2_IN
- net bit1_in renamed BIT1_IN
- net bit3_in renamed BIT3_IN
- net c: no longer names the net of DS1.7 (c), RN2.6 (R6.1)
- net d: no longer names the net of DS1.5 (d), RN2.5 (R5.1)
- net dp: no longer names the net of DS1.6 (DP), RN2.1 (R1.1)
- net e: no longer names the net of DS1.4 (e), RN2.4 (R4.1)
- net f: no longer names the net of DS1.2 (f), RN2.3 (R3.1)
- net g: no longer names the net of DS1.1 (g), RN2.2 (R2.1)
Other:
- note added: "M5_NibbleToHex_ver01, 25 August 2026 Tamanna Chadak, Tobe Cynar, Baird Soules umassamherstm5.org/........."
- moved on the sheet: DS1, RN2

Commit message: PCB RevA
Parts:
- added C1: 0.1µF, symbol Device:C
Connections:
- net +5V: no longer IC1.24 (VCC)
- net GND: now also C1.2
- net BIT1_IN renamed D1
- net BIT2_IN renamed D0
- net D0: no longer IC1.3 (IN_2), J1.4 (Pin_4), RN1.3 (R2)
- net BIT3_IN renamed D3
- net BLANK_IN_N renamed BLANK_N
- net DP_IN renamed DP
- new net: C1.1, IC1.24 (VCC)
- new net D2: IC1.3 (IN_2), J1.4 (Pin_4), RN1.3 (R2)
Other:
- note added: "M5_NibbleToHex_ver0.6, 8 September 2026 Tamanna Chadak, Tobe Cynar, Baird Soules umassamherstm5.org/........."
- note removed: "M5_NibbleToHex_ver01, 25 August 2026 Tamanna Chadak, Tobe Cynar, Baird Soules umassamherstm5.org/........."
- moved on the sheet: J1, RN1

Commit message: v0.5
Parts:
- added D1, D2, D3, D4: LED, LED_THT:LED_D3.0mm, symbol Device:LED
- added RN2: 330, Package_DIP:DIP-8_W7.62mm, symbol Device:R_Pack04
- C1: footprint (none) -> Capacitor_THT:C_Disc_D5.0mm_W2.5mm_P2.50mm
- RN1: value 12K -> 10K
- renumbered RN2 to RN3
Connections:
- net +5V: now also C1.1, IC1.24 (VCC)
- net D0: now also RN2.1 (R1.1)
- net D1: now also RN2.2 (R2.1)
- net D2: now also RN2.3 (R3.1)
- net D3: now also RN2.4 (R4.1)
- net GND: now also D1.2 (A), D2.2 (A), D3.2 (A), D4.2 (A)
- new net: D3.1 (K), RN2.6 (R3.2)
- new net: D2.1 (K), RN2.7 (R2.2)
- new net: D4.1 (K), RN2.5 (R4.2)
- new net: D1.1 (K), RN2.8 (R1.2)
Other:
- note added: "M5_NibbleToHex_RevB, 24 September 2026 Tamanna Chadak, Tobe Cynar, Baird Soules https://www.umassamherstm5.org/blog/m5hexdisplay"
- note removed: "M5_NibbleToHex_ver0.6, 8 September 2026 Tamanna Chadak, Tobe Cynar, Baird Soules umassamherstm5.org/........."
- moved on the sheet: C1, DS1, IC1, J1, RN1, RN3

Commit message: RevB updates
Parts:
- removed RN2: 330, Package_DIP:DIP-8_W7.62mm, symbol Device:R_Pack04
- added R1, R2, R3, R4: 330, Resistor_THT:R_Axial_DIN0207_L6.3mm_D2.5mm_P7.62mm_Horizontal, symbol Device:R_US
- renumbered RN3 to RN2
Connections:
- net D0: now also R1.1
- net D1: now also R2.1
- net D2: now also R3.1
- net D3: now also R4.1
- net at D3.1 (K): now also R3.2
- net at D2.1 (K): now also R2.2
- net at D4.1 (K): now also R4.2
- net at D1.1 (K): now also R1.2

Commit message: Rev B
Connections:
- net GND: now also D1.1 (K), D2.1 (K), D3.1 (K), D4.1 (K); no longer D1.2 (A), D2.2 (A), D3.2 (A), D4.2 (A)
- net at R3.2: now also D3.2 (A); no longer D3.1 (K)
- net at R2.2: now also D2.2 (A); no longer D2.1 (K)
- net at R4.2: now also D4.2 (A); no longer D4.1 (K)
- net at R1.2: now also D1.2 (A); no longer D1.1 (K)
Other:
- note added: "M5_NibbleToHex_RevB, 29 September 2026 Tamanna Chadak, Tobe Cynar, Baird Soules https://www.umassamherstm5.org/blog/m5hexdisplay"
- note removed: "M5_NibbleToHex_RevB, 24 September 2026 Tamanna Chadak, Tobe Cynar, Baird Soules https://www.umassamherstm5.org/blog/m5hexdisplay"
- moved on the sheet: D1, D2, D3, D4

Commit message: Rev B
Parts:
- IC1: footprint Package_DIP:DIP-24_W10.16mm -> Package_DIP:DIP-24_W7.62mm
Changed lines of the file:
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@@
 			)
 		)
-		(property "Footprint" "Package_DIP:DIP-24_W10.16mm"
+		(property "Footprint" "Package_DIP:DIP-24_W7.62mm"
 			(at 138.43 202.87 0)
 			(hide yes)
