File: CPLD_bcdtohex.kicad_pcb (KiCad board)
At the start: 2 copper layers, 27 x 90.1 mm, 6 parts, among them IC1 ATF750C-10PU, J1 Conn_01x06, J2 Conn_01x02

Commit message: Initial commit
Parts:
- removed J2: Conn_01x02, Connector_PinHeader_2.54mm:PinHeader_1x02_P2.54mm_Vertical
- J1: value Conn_01x06 -> Conn_01x08_Pin; footprint Connector_PinHeader_2.54mm:PinHeader_1x06_P2.54mm_Vertical -> Connector_PinHeader_2.54mm:PinHeader_1x08_P2.54mm_Vertical
- moved J1 6.42 mm to (143.9, 148.7)
Connections:
- net /a renamed Net-(DS1-a)
- net /b renamed Net-(DS1-b)
- net /c renamed Net-(DS1-c)
- net /d renamed Net-(DS1-d)
- net /dp renamed Net-(DS1-DP)
- net /e renamed Net-(DS1-e)
- net /f renamed Net-(DS1-f)
- net /g renamed Net-(DS1-g)
- net Net-(IC1-I/O_1) renamed /DP_OUT_N
- net Net-(IC1-I/O_2) renamed /SEG_G_OUT_N
- net Net-(IC1-I/O_3) renamed /SEG_F_OUT_N
- net Net-(IC1-I/O_4) renamed /SEG_E_OUT_N
- net Net-(IC1-I/O_5) renamed /SEG_D_OUT_N
- net Net-(IC1-I/O_6) renamed /SEG_C_OUT_N
- net Net-(IC1-I/O_7) renamed /SEG_B_OUT_N
- net Net-(IC1-I/O_8) renamed /SEG_A_OUT_N
- IC1 pad 2: /bit3_in -> /BIT3_IN
- IC1 pad 3: /bit2_in -> /BIT2_IN
- IC1 pad 4: /bit1_in -> /BIT1_IN
- IC1 pad 5: /bit0_in -> /BIT2_IN
- IC1 pad 6: /BLANK_in -> /BLANK_IN_N
- IC1 pad 7: /DP_in -> /DP_IN
- J1 pad 1: /bit3_in -> +5V
- J1 pad 2: /bit2_in -> GND
- J1 pad 3: /bit1_in -> /BIT3_IN
- J1 pad 4: /bit0_in -> /BIT2_IN
- J1 pad 5: /BLANK_in -> /BIT1_IN
- J1 pad 6: /DP_in -> /BIT2_IN
- RN1 pad 2: /bit3_in -> /BIT3_IN
- RN1 pad 3: /bit2_in -> /BIT2_IN
- RN1 pad 4: /bit1_in -> /BIT1_IN
- RN1 pad 5: /bit0_in -> /BIT2_IN
- RN1 pad 6: /BLANK_in -> /BLANK_IN_N
- RN1 pad 7: /DP_in -> /DP_IN
Routing:
- net /BIT2_IN: track 0.00 -> 75.6 mm
- net /bit3_in: track 41.4 -> 0.00 mm
- net /BIT3_IN: track 0.00 -> 41.0 mm
- net /DP_in: track 40.4 -> 0.00 mm
- net /DP_IN: track 0.00 -> 40.1 mm
- net /bit2_in: track 39.5 -> 0.00 mm
- net /bit1_in: track 37.7 -> 0.00 mm
- net /BIT1_IN: track 0.00 -> 37.4 mm
- net /bit0_in: track 36.8 -> 0.00 mm
- net /BLANK_in: track 33.2 -> 0.00 mm
- net /BLANK_IN_N: track 0.00 -> 32.8 mm
Other:
- board text added: "+5V"
- board text added: "BIT0_IN"
- board text added: "BIT1_IN"
- board text added: "BIT2_IN"
- board text added: "BIT3_IN"
- board text added: "BLANK_IN_N"
- board text added: "COMMON ANODE"
- board text added: "DP_IN"
- board text added: "M5_NibbleToHex_ver01, 25 August 2026 Tamanna Chandak, Tobe Cynar, Baird Soules"
- board text added: "SEG_A"
- board text added: "SEG_B"
- board text added: "SEG_C"
- board text added: "SEG_D"
- board text added: "SEG_DP"
- board text added: "SEG_E"
- board text added: "SEG_F"
- board text added: "SEG_G"
- board text removed: "5V"
- board text removed: "Seeing the Nibble: A Breadboard-Friendly Hexadecimal Display for Teaching Digital Logic and Programmable Hardware"
- board text removed: "bit0 (2^0)"
- board text removed: "bit1 (2^1)"
- board text removed: "bit2 (2^2)"
- board text removed: "bit3 (2^3)"
- board text removed: "blanking"
- board text removed: "common anode"
- board text removed: "decimal point"
- board text removed: "seg_a"
- board text removed: "seg_b"
- board text removed: "seg_c"
- board text removed: "seg_d"
- board text removed: "seg_dp"
- board text removed: "seg_e"
- board text removed: "seg_f"
- board text removed: "seg_g"
