File: CPLD_bcdtohex.kicad_pcb (KiCad board)
At the start: 2 copper layers, 27 x 90.1 mm, 5 parts, among them IC1 ATF750C-10PU, J1 Conn_01x08_Pin

Commit message: PCB RevA
Parts:
- added C1: 0.1µF, Capacitor_THT:C_Disc_D10.0mm_W2.5mm_P5.00mm, F.Cu at (163.5, 114.5)
- added mh: MountingHole_2.7mm_M2.5, MountingHole:MountingHole_2.7mm_M2.5, F.Cu at (163.0, 138.0)
- added mh: MountingHole_2.7mm_M2.5, MountingHole:MountingHole_2.7mm_M2.5, F.Cu at (141.5, 63.0)
Connections:
- net /BIT1_IN renamed /D1
- net /BIT3_IN renamed /D3
- net /BLANK_IN_N renamed /BLANK
- net /DP_IN renamed /DP
- IC1 pad 24: +5V -> Net-(IC1-VCC)
- IC1 pad 3: /BIT2_IN -> /D2
- IC1 pad 5: /BIT2_IN -> /D0
- J1 pad 4: /BIT2_IN -> /D2
- J1 pad 6: /BIT2_IN -> /D0
- RN1 pad 3: /BIT2_IN -> /D2
- RN1 pad 5: /BIT2_IN -> /D0
Routing:
- net /BIT2_IN: track 75.6 -> 0.00 mm
- net /D2: track 0.00 -> 39.2 mm
- net /D0: track 0.00 -> 36.4 mm
- net Net-(IC1-VCC): track 0.00 -> 8.93 mm
- added copper zone on In1.Cu, net +5V
- added copper zone on In2.Cu, net GND
- removed copper zone on F.Cu, net +5V
- removed copper zone on B.Cu, net GND
Other:
- board size 27 x 90.1 mm -> 30.5 x 96 mm
- copper layers 2 -> 4
- board text added: "BL_N"
- board text added: "CA"
- board text added: "D0"
- board text added: "D1"
- board text added: "D2"
- board text added: "D3"
- board text added: "DP"
- board text added: "M5_NibbleToHex_REV A, 9 September 2026 Tamanna Chandak, Tobe Cynar, Baird Soules"
- board text added: "https://www.umassamherstm5.org/blog/m5hexdisplay"
- board text removed: "BIT0_IN"
- board text removed: "BIT1_IN"
- board text removed: "BIT2_IN"
- board text removed: "BIT3_IN"
- board text removed: "BLANK_IN_N"
- board text removed: "COMMON ANODE"
- board text removed: "DP_IN"
- board text removed: "M5_NibbleToHex_ver01, 25 August 2026 Tamanna Chandak, Tobe Cynar, Baird Soules"

Commit message: v0.5
Parts:
- removed mh (x2): MountingHole_2.7mm_M2.5, MountingHole:MountingHole_2.7mm_M2.5
- added D1: LED, LED_THT:LED_D3.0mm, F.Cu at (140.5, 66.0)
- added D2: LED, LED_THT:LED_D3.0mm, F.Cu at (135.0, 66.0)
- added D3: LED, LED_THT:LED_D3.0mm, F.Cu at (129.5, 66.0)
- added D4: LED, LED_THT:LED_D3.0mm, F.Cu at (124.0, 66.0)
- added RN3: 330, Package_DIP:DIP-16_W7.62mm, F.Cu at (129.7, 74.1)
- C1: footprint Capacitor_THT:C_Disc_D10.0mm_W2.5mm_P5.00mm -> Capacitor_THT:C_Disc_D5.0mm_W2.5mm_P2.50mm
- RN1: value 12K -> 10K
- RN2: value 330 -> 220; footprint Package_DIP:DIP-16_W7.62mm -> Package_DIP:DIP-8_W7.62mm
- moved RN2 68.4 mm to (129.7, 148.3), turned to 90 degrees
- moved C1 35.1 mm to (132.2, 98.5), turned to 0 degrees
- moved DS1 26.0 mm to (130.0, 47.4)
- moved J1 22.2 mm to (124.3, 159.0)
- moved RN1 22.0 mm to (125.4, 154.0)
- moved IC1 19.1 mm to (128.3, 106.4)
Connections:
- net /BLANK renamed /BLANK_N
- C1 pad 1: Net-(IC1-VCC) -> +5V
- IC1 pad 24: Net-(IC1-VCC) -> +5V
- RN2 pad 1: Net-(DS1-DP) -> /D0
- RN2 pad 2: Net-(DS1-g) -> /D1
- RN2 pad 3: Net-(DS1-f) -> /D2
- RN2 pad 4: Net-(DS1-e) -> /D3
- RN2 pad 5: Net-(DS1-d) -> Net-(D4-K)
- RN2 pad 6: Net-(DS1-c) -> Net-(D3-K)
- RN2 pad 7: Net-(DS1-b) -> Net-(D2-K)
- RN2 pad 8: Net-(DS1-a) -> Net-(D1-K)
Routing:
- net Net-(D1-K): track 0.00 -> 118.0 mm
- net Net-(D2-K): track 0.00 -> 113.4 mm
- net Net-(D3-K): track 0.00 -> 97.9 mm
- net Net-(D4-K): track 0.00 -> 85.4 mm
- net Net-(DS1-b): track 38.6 -> 104.2 mm
- net Net-(DS1-c): track 26.3 -> 88.7 mm
- net /D0: track 36.4 -> 67.8 mm
- net /D3: track 41.0 -> 71.2 mm
- net /D1: track 37.4 -> 63.0 mm
- net Net-(DS1-DP): track 10.5 -> 31.5 mm
- net /D2: track 39.2 -> 58.7 mm
- net /BLANK_N: track 32.8 -> 51.5 mm
- net Net-(DS1-g): track 20.6 -> 37.6 mm
- net Net-(DS1-d): track 19.0 -> 31.2 mm
- net Net-(DS1-f): track 21.6 -> 32.0 mm
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- added copper zone on F.Cu, net +5V
- removed copper zone on In1.Cu, net +5V
Other:
- board size 30.5 x 96 mm -> 31.5 x 122.8 mm
- board text added: "Binary"
- board text added: "Hexadecimal"
- board text added: "M5_NibbleToHex_REV B, 28 September 2026 Tamanna Chandak, Tobe Cynar, Baird Soules"
- board text removed: "+5V"
- board text removed: "7 Segment Display"
- board text removed: "M5_NibbleToHex_REV A, 9 September 2026 Tamanna Chandak, Tobe Cynar, Baird Soules"
- board text removed: "SEG_B"

Commit message: RevB updates
Parts:
- removed the RN2 at (129.7, 148.3)
- added R1: 330, Resistor_THT:R_Axial_DIN0207_L6.3mm_D2.5mm_P7.62mm_Horizontal, F.Cu at (139.0, 148.4)
- added R2: 330, Resistor_THT:R_Axial_DIN0207_L6.3mm_D2.5mm_P7.62mm_Horizontal, F.Cu at (135.0, 148.3)
- added R3: 330, Resistor_THT:R_Axial_DIN0207_L6.3mm_D2.5mm_P7.62mm_Horizontal, F.Cu at (131.2, 148.4)
- added R4: 330, Resistor_THT:R_Axial_DIN0207_L6.3mm_D2.5mm_P7.62mm_Horizontal, F.Cu at (127.5, 148.4)
- renumbered RN3 to RN2
Routing:
- net Net-(D1-K): track 118.0 -> 97.5 mm
- net Net-(D2-K): track 113.4 -> 93.3 mm
- net /D2: track 58.7 -> 78.1 mm
- net /D1: track 63.0 -> 76.8 mm
- net /BLANK_N: track 51.5 -> 61.3 mm
- net /DP: track 49.4 -> 57.2 mm
- net /D0: track 67.8 -> 75.3 mm
- net /D3: track 71.2 -> 78.2 mm
- net Net-(D3-K): track 97.9 -> 92.2 mm
- net Net-(DS1-DP): track 31.5 -> 34.0 mm
- net Net-(D4-K): track 85.4 -> 84.5 mm

Commit message: Rev B
Connections:
- D1 pad 1: Net-(D1-K) -> GND
- D1 pad 2: GND -> Net-(D1-A)
- D2 pad 1: Net-(D2-K) -> GND
- D2 pad 2: GND -> Net-(D2-A)
- D3 pad 1: Net-(D3-K) -> GND
- D3 pad 2: GND -> Net-(D3-A)
- D4 pad 1: Net-(D4-K) -> GND
- D4 pad 2: GND -> Net-(D4-A)
- R1 pad 2: Net-(D1-K) -> Net-(D1-A)
- R2 pad 2: Net-(D2-K) -> Net-(D2-A)
- R3 pad 2: Net-(D3-K) -> Net-(D3-A)
- R4 pad 2: Net-(D4-K) -> Net-(D4-A)
Routing:
- net Net-(D1-K): track 97.5 -> 0.00 mm
- net Net-(D1-A): track 0.00 -> 97.5 mm
- net Net-(D2-K): track 93.3 -> 0.00 mm
- net Net-(D3-K): track 92.2 -> 0.00 mm
- net Net-(D2-A): track 0.00 -> 90.6 mm
- net Net-(D4-K): track 84.5 -> 0.00 mm
- net Net-(D3-A): track 0.00 -> 81.0 mm
- net Net-(D4-A): track 0.00 -> 77.2 mm
Other:
- board text added: "M5_NibbleToHex_REV B, 29 September 2026 Tamanna Chandak, Tobe Cynar, Baird Soules"
- board text removed: "M5_NibbleToHex_REV B, 28 September 2026 Tamanna Chandak, Tobe Cynar, Baird Soules"
Changed lines of the file:
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@@
 			(layers "*.Cu" "*.Mask")
 			(remove_unused_layers no)
-			(net "Net-(D3-K)")
+			(net "GND")
 			(pinfunction "K_1")
 			(pintype "passive")
@@
 			(layers "*.Cu" "*.Mask")
 			(remove_unused_layers no)
-			(net "GND")
+			(net "Net-(D3-A)")
 			(pinfunction "A_2")
 			(pintype "passive")
@@
 			(layers "*.Cu" "*.Mask")
 			(remove_unused_layers no)
-			(net "Net-(D4-K)")
+			(net "Net-(D4-A)")
 			(pintype "passive")
 		)
@@
 			(layers "*.Cu" "*.Mask")
 			(remove_unused_layers no)
-			(net "Net-(D1-K)")
+			(net "GND")
 			(pinfunction "K_1")
 			(pintype "passive")
@@
 			(layers "*.Cu" "*.Mask")
 			(remove_unused_layers no)
-			(net "GND")
+			(net "Net-(D1-A)")
 			(pinfunction "A_2")
 			(pintype "passive")
@@
 			(layers "*.Cu" "*.Mask")
 			(remove_unused_layers no)
-			(net "Net-(D4-K)")
+			(net "GND")
 			(pinfunction "K_1")
 			(pintype "passive")
@@
 			(layers "*.Cu" "*.Mask")
 			(remove_unused_layers no)
-			(net "GND")
+			(net "Net-(D4-A)")
 			(pinfunction "A_2")
 			(pintype "passive")
@@
 			(layers "*.Cu" "*.Mask")
 			(remove_unused_layers no)
-			(net "Net-(D3-K)")
+			(net "Net-(D3-A)")
 			(pintype "passive")
 		)
@@
 			(layers "*.Cu" "*.Mask")
 			(remove_unused_layers no)
-			(net "Net-(D2-K)")
+			(net "Net-(D2-A)")
 			(pintype "passive")
 		)
@@
 			(layers "*.Cu" "*.Mask")
 			(remove_unused_layers no)
-			(net "Net-(D1-K)")
+			(net "Net-(D1-A)")
 			(pintype "passive")
 		)
@@
 			(layers "*.Cu" "*.Mask")
 			(remove_unused_layers no)
-			(net "Net-(D2-K)")
+			(net "GND")
 			(pinfunction "K_1")
 			(pintype "passive")
@@
 			(layers "*.Cu" "*.Mask")
 			(remove_unused_layers no)
-			(net "GND")
+			(net "Net-(D2-A)")
 			(pinfunction "A_2")
 			(pintype "passive")
@@
 		)
 	)
-	(gr_text "M5_NibbleToHex_REV B, 28 September 2026\nTamanna Chandak, Tobe Cynar, Baird Soules"
+	(gr_text "M5_NibbleToHex_REV B, 29 September 2026\nTamanna Chandak, Tobe Cynar, Baird Soules"
 		(at 123 144.5 90)
 		(layer "F.SilkS")
@@
 	)
 	(segment
-		(start 126.5 69)
-		(end 129.5 66)
-		(width 0.2)
-		(layer "F.Cu")
-		(net "Net-(D3-K)")
-	)
-	(segment
-		(start 129.5 139)
-		(end 126.75 139)
-		(width 0.2)
-		(layer "F.Cu")
-		(net "Net-(D3-K)")
-	)
-	(segment
-		(start 126.75 139)
-		(end 116.25 128.5)
+		(start 132.04 66)
+		(end 124.85 73.19)
 		(width 0.2)
 		(layer "F.Cu")
-		(net "Net-(D3-K)")
+		(net "Net-(D3-A)")
 	)
 	(segment
-		(start 119.5 69)
-		(end 126.5 69)
+		(start 128.118629 138.75)
+		(end 129.25 138.75)
 		(width 0.2)
 		(layer "F.Cu")
-		(net "Net-(D3-K)")
+		(net "Net-(D3-A)")
 	)
 	(segment
-		(start 116.25 72.25)
-		(end 119.5 69)
+		(start 124.85 135.481371)
+		(end 128.118629 138.75)
 		(width 0.2)
 		(layer "F.Cu")
-		(net "Net-(D3-K)")
+		(net "Net-(D3-A)")
 	)
 	(segment
-		(start 131.25 140.75)
-		(end 129.5 139)
+		(start 124.85 73.19)
+		(end 124.85 135.481371)
 		(width 0.2)
 		(layer "F.Cu")
-		(net "Net-(D3-K)")
+		(net "Net-(D3-A)")
 	)
 	(segment
-		(start 116.25 128.5)
-		(end 116.25 72.25)
+		(start 129.25 138.75)
+		(end 131.25 140.75)
 		(width 0.2)
 		(layer "F.Cu")
-		(net "Net-(D3-K)")
+		(net "Net-(D3-A)")
 	)
 	(segment
@@
 	)
 	(segment
-		(start 121.5 66)
-		(end 115.75 71.75)
+		(start 124 68.5)
+		(end 126.5 66)
 		(width 0.2)
 		(layer "F.Cu")
-		(net "Net-(D4-K)")
+		(net "Net-(D4-A)")
 	)
 	(segment
-		(start 115.75 129)
-		(end 115.75 71.75)
-		(width 0.2)
-		(layer "F.Cu")
-		(net "Net-(D4-K)")
-	)
-	(segment
-		(start 123.96 66)
-		(end 121.5 66)
+		(start 127.5 140.75)
+		(end 124 137.25)
 		(width 0.2)
 		(layer "F.Cu")
-		(net "Net-(D4-K)")
+		(net "Net-(D4-A)")
 	)
 	(segment
-		(start 127.5 140.75)
-		(end 115.75 129)
+		(start 124 137.25)
+		(end 124 68.5)
 		(width 0.2)
 		(layer "F.Cu")
-		(net "Net-(D4-K)")
+		(net "Net-(D4-A)")
 	)
 	(segment
-		(start 124.25 72.75)
-		(end 125.25 71.75)
+		(start 126.75 74.5)
+		(end 126.75 136.25)
 		(width 0.2)
 		(layer "F.Cu")
-		(net "Net-(D1-K)")
+		(net "Net-(D1-A)")
 	)
 	(segment
-		(start 127 136.25)
-		(end 124.25 133.5)
+		(start 134.5 136.25)
+		(end 139 140.75)
 		(width 0.2)
 		(layer "F.Cu")
-		(net "Net-(D1-K)")
+		(net "Net-(D1-A)")
 	)
 	(segment
-		(start 125.25 71.75)
-		(end 134.71 71.75)
+		(start 129.782843 71.467157)
+		(end 126.75 74.5)
 		(width 0.2)
 		(layer "F.Cu")
-		(net "Net-(D1-K)")
+		(net "Net-(D1-A)")
 	)
 	(segment
-		(start 134.5 136.25)
-		(end 127 136.25)
+		(start 140.717157 71.467157)
+		(end 129.782843 71.467157)
 		(width 0.2)
 		(layer "F.Cu")
-		(net "Net-(D1-K)")
+		(net "Net-(D1-A)")
 	)
 	(segment
-		(start 139 140.75)
+		(start 126.75 136.25)
 		(end 134.5 136.25)
 		(width 0.2)
 		(layer "F.Cu")
-		(net "Net-(D1-K)")
+		(net "Net-(D1-A)")
 	)
 	(segment
-		(start 134.71 71.75)
-		(end 140.46 66)
+		(start 143 66)
+		(end 143 69.184314)
 		(width 0.2)
 		(layer "F.Cu")
-		(net "Net-(D1-K)")
+		(net "Net-(D1-A)")
 	)
 	(segment
-		(start 124.25 133.5)
-		(end 124.25 72.75)
+		(start 143 69.184314)
+		(end 140.717157 71.467157)
 		(width 0.2)
 		(layer "F.Cu")
-		(net "Net-(D1-K)")
+		(net "Net-(D1-A)")
 	)
 	(segment
@@
 	)
 	(segment
-		(start 119.5 76.934314)
-		(end 119.5 130.5)
+		(start 137.5 69.25)
+		(end 137.5 66)
+		(width 0.2)
+		(layer "F.Cu")
+		(net "Net-(D2-A)")
+	)
+	(segment
+		(start 125.25 135.315685)
+		(end 125.25 74.25)
 		(width 0.2)
 		(layer "F.Cu")
-		(net "Net-(D2-K)")
+		(net "Net-(D2-A)")
 	)
 	(segment
-		(start 129.61 71.35)
-		(end 125.084314 71.35)
+		(start 125.25 74.25)
+		(end 129.75 69.75)
 		(width 0.2)
 		(layer "F.Cu")
-		(net "Net-(D2-K)")
+		(net "Net-(D2-A)")
 	)
 	(segment
-		(start 125.084314 71.35)
-		(end 119.5 76.934314)
+		(start 129.75 69.75)
+		(end 137 69.75)
 		(width 0.2)
 		(layer "F.Cu")
-		(net "Net-(D2-K)")
+		(net "Net-(D2-A)")
 	)
 	(segment
-		(start 126.5 137.5)
-		(end 131.81 137.5)
+		(start 130.96 136.65)
+		(end 126.584315 136.65)
 		(width 0.2)
 		(layer "F.Cu")
-		(net "Net-(D2-K)")
+		(net "Net-(D2-A)")
 	)
 	(segment
-		(start 131.81 137.5)
-		(end 135 140.69)
+		(start 137 69.75)
+		(end 137.5 69.25)
 		(width 0.2)
 		(layer "F.Cu")
-		(net "Net-(D2-K)")
+		(net "Net-(D2-A)")
 	)
 	(segment
-		(start 134.96 66)
-		(end 129.61 71.35)
+		(start 135 140.69)
+		(end 130.96 136.65)
 		(width 0.2)
 		(layer "F.Cu")
-		(net "Net-(D2-K)")
+		(net "Net-(D2-A)")
 	)
 	(segment
-		(start 119.5 130.5)
-		(end 126.5 137.5)
+		(start 126.584315 136.65)
+		(end 125.25 135.315685)
 		(width 0.2)
 		(layer "F.Cu")
-		(net "Net-(D2-K)")
+		(net "Net-(D2-A)")
 	)
 	(zone

Commit message: Rev B
Parts:
- IC1: footprint Package_DIP:DIP-24_W10.16mm -> Package_DIP:DIP-24_W7.62mm
- moved IC1 1.16 mm to (129.5, 106.4)
Routing:
- net /DP_OUT_N: track 59.1 -> 62.7 mm
- net /SEG_C_OUT_N: track 34.7 -> 36.1 mm
- net /SEG_G_OUT_N: track 56.8 -> 58.1 mm
- net /SEG_F_OUT_N: track 51.4 -> 52.7 mm
- net /SEG_E_OUT_N: track 45.8 -> 47.2 mm
- net /SEG_D_OUT_N: track 40.4 -> 41.7 mm
- net /SEG_B_OUT_N: track 29.3 -> 30.7 mm
- net /SEG_A_OUT_N: track 23.9 -> 25.3 mm
- net /D0: track 75.3 -> 76.5 mm
- net /DP: track 57.2 -> 58.4 mm
- net /D3: track 78.2 -> 79.4 mm
- net /D1: track 76.8 -> 78.0 mm
- net /BLANK_N: track 61.3 -> 62.5 mm
- net /D2: track 78.1 -> 79.3 mm
